File: circuit/7-seg-array-clock.kicad_pcb (KiCad board)
At the start: 2 copper layers, 304.8 x 114.3 mm, 91 parts, among them U1 CC56-12EWA, U10 CC56-12EWA, U11 CC56-12EWA, U12 MAX7219, U13 CC56-12EWA, U14 CC56-12EWA, U15 MAX7219, U16 CC56-12EWA, U17 CC56-12EWA, U18 MAX7219, U19 CC56-12EWA, U2 MAX7219, U20 CC56-12EWA, U21 MAX7219, U22 CC56-12EWA, U23 CC56-12EWA, U24 MAX7219, U25 CC56-12EWA, U26 CC56-12EWA, U27 MAX7219, U28 CC56-12EWA, U29 CC56-12EWA, U3 CC56-12EWA, U30 MAX7219, U31 CC56-12EWA, U32 CC56-12EWA, U33 MAX7219, U34 CC56-12EWA, U35 CC56-12EWA, U36 MAX7219, U37 CC56-12EWA, U38 CC56-12EWA, U39 MAX7219, U4 CC56-12EWA, U40 CC56-12EWA, U41 CC56-12EWA, U42 MAX7219, U43 CC56-12EWA, U44 CC56-12EWA, U45 MAX7219, U46 CC56-12EWA, U47 CC56-12EWA, U48 MAX7219, U49 CC56-12EWA, U5 MAX7219, U50 CC56-12EWA, U51 MAX7219, U52 CC56-12EWA, U53 CC56-12EWA, U54 MAX7219, U55 CC56-12EWA, U6 CC56-12EWA, U7 ESP-12F, U8 CC56-12EWA, U9 MAX7219

Commit message: Added tracks to first display
Parts:
- moved R1 0.24 mm to (15.2, -170.2)
Routing:
- net +5V: track 0.00 -> 305.6 mm, vias 0 -> 2
- net /display0/G: track 0.00 -> 82.4 mm
- net /display0/DP: track 0.00 -> 81.6 mm
- net /display0/A: track 0.00 -> 78.2 mm
- net /display0/C: track 0.00 -> 77.0 mm, vias 0 -> 1
- net /display0/D: track 0.00 -> 76.6 mm
- net /display0/E: track 0.00 -> 74.0 mm, vias 0 -> 1
- net /display0/B: track 0.00 -> 72.4 mm
- net /display0/F: track 0.00 -> 55.7 mm, vias 0 -> 1
- net /display0/D0: track 0.00 -> 54.7 mm
- net /display0/D6: track 0.00 -> 44.7 mm
- net /display0/D5: track 0.00 -> 39.2 mm, vias 0 -> 1
- net /display0/D7: track 0.00 -> 37.4 mm
- net /display0/D1: track 0.00 -> 34.2 mm
- net /display0/D2: track 0.00 -> 33.2 mm
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Other:
- net class Power added: clearance 0.2, trace_width 0.5, via_dia 0.8, via_drill 0.4

Commit message: Routed all displays
Parts:
- U7: moved to B.Cu
- moved U7 338.0 mm to (66.0, -160.1), turned to 180 degrees
- moved U35 50.8 mm to (186.7, -97.8)
- moved U37 50.8 mm to (237.5, -97.8)
- moved U44 50.8 mm to (186.7, -78.7)
- moved U46 50.8 mm to (237.5, -78.7)
- moved U20 50.8 mm to (-16.5, -116.8)
- moved U22 50.8 mm to (34.3, -116.8)
- moved U29 50.8 mm to (-16.5, -97.8)
- moved U31 50.8 mm to (34.3, -97.8)
- moved U47 50.8 mm to (-16.5, -59.7)
- moved U49 50.8 mm to (34.3, -59.7)
- moved R4 20.4 mm to (15.2, -151.1)
- moved R10 18.8 mm to (15.2, -113.2)
- moved R5 17.9 mm to (116.8, -151.1)
- moved R7 16.1 mm to (15.2, -132.2)
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Routing:
- net GND: track 8.09 -> 145.6 mm, vias 3 -> 57
- net /display5/G: track 0.00 -> 82.5 mm
- net /display14/G: track 0.00 -> 82.5 mm
- net /display6/G: track 0.00 -> 82.5 mm
- net /display4/G: track 0.00 -> 82.5 mm
- net /display17/G: track 0.00 -> 82.5 mm
- net /display15/G: track 0.00 -> 82.5 mm
- net /display13/G: track 0.00 -> 82.5 mm
- net /display3/G: track 0.00 -> 82.5 mm
- net /display18/G: track 0.00 -> 82.5 mm
- net /display16/G: track 0.00 -> 82.5 mm
- net /display11/G: track 0.00 -> 82.5 mm
- net /display1/G: track 0.00 -> 82.5 mm
- net /display8/G: track 0.00 -> 82.5 mm
- net /display9/G: track 0.00 -> 82.5 mm
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Other:
- board size 304.8 x 114.3 mm -> 304.8 x 115.6 mm

Commit message: Updated display footprint
Other:
- board outline removed

Commit message: Fixed display clearance issues
Parts:
- moved C18 2.54 mm to (228.6, -64.8)
- moved R16 2.54 mm to (15.2, -72.5)
- moved R17 2.54 mm to (116.8, -72.5)
- moved R18 2.54 mm to (218.4, -72.4)
- moved U48 2.54 mm to (15.2, -64.8)
- moved U51 2.54 mm to (116.8, -64.8)
- moved U54 2.54 mm to (218.4, -64.8)
- moved U47 2.54 mm to (-16.5, -57.1)
- moved U49 2.54 mm to (34.3, -57.1)
- moved U50 2.54 mm to (85.1, -57.1)
- moved U52 2.54 mm to (135.9, -57.1)
- moved U53 2.54 mm to (186.7, -57.1)
- moved U55 2.54 mm to (237.5, -57.1)
- moved C16 2.54 mm to (25.4, -65.0)
- moved C17 2.54 mm to (127.0, -65.0)
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
Commit message: Updated footprint to the proper one
Parts:
- U1, U10, U11, U13, U14, U16, U17, U19, U20, U22, U23, U25, U26, U28, U29, U3, U31, U32, U34, U35, U37, U38, U4, U40, U41, U43, U44, U46, U47, U49, U50, U52, U53, U55, U6, U8: footprint Display_7Segment:CA56-12EWA -> circuit:7seg
Routing:
- net /display0/D0: track 54.7 -> 53.8 mm
- net /display1/D0: track 54.7 -> 53.8 mm
- net /display3/D0: track 54.7 -> 53.8 mm
Other:
- board outline added: 304.8 x 117.3 mm

Commit message: Added controller to PCB
Parts:
- added C19: 10µF, Capacitor_SMD:C_0805_2012Metric_Pad1.15x1.40mm_HandSolder, B.Cu at (57.8, -121.3)
- added C20: 10µF, Capacitor_SMD:C_0805_2012Metric_Pad1.15x1.40mm_HandSolder, B.Cu at (57.8, -117.2)
- added J1: FTDI, Connector_PinHeader_2.54mm:PinHeader_1x04_P2.54mm_Vertical, B.Cu at (62.2, -135.9)
- added R19: 10k, Resistor_SMD:R_0805_2012Metric_Pad1.15x1.40mm_HandSolder, B.Cu at (80.0, -150.7)
- added R20: 10k, Resistor_SMD:R_0805_2012Metric_Pad1.15x1.40mm_HandSolder, B.Cu at (77.5, -150.7)
- added R21: 10k, Resistor_SMD:R_0805_2012Metric_Pad1.15x1.40mm_HandSolder, B.Cu at (70.7, -139.7)
- added R22: 10k, Resistor_SMD:R_0805_2012Metric_Pad1.15x1.40mm_HandSolder, B.Cu at (54.6, -150.5)
- added SW1: Reset, Button_Switch_SMD:SW_SPST_CK_RS282G05A3, B.Cu at (81.3, -163.8)
- added SW2: Flash, Button_Switch_SMD:SW_SPST_CK_RS282G05A3, B.Cu at (66.0, -143.5)
- added U56: LM1117-3.3, Package_TO_SOT_SMD:SOT-223-3_TabPin2, B.Cu at (66.0, -119.4)
Connections:
- U12 pad 12: /display4/LOAD -> LOAD
- U12 pad 13: /display4/CLK -> CLK
- U15 pad 12: /display5/LOAD -> LOAD
- U15 pad 13: /display5/CLK -> CLK
- U18 pad 12: /display6/LOAD -> LOAD
- U18 pad 13: /display6/CLK -> CLK
- U2 pad 12: /display0/LOAD -> LOAD
- U2 pad 13: /display0/CLK -> CLK
- U21 pad 12: /display7/LOAD -> LOAD
- U21 pad 13: /display7/CLK -> CLK
- U24 pad 12: /display8/LOAD -> LOAD
- U24 pad 13: /display8/CLK -> CLK
- U27 pad 12: /display9/LOAD -> LOAD
- U27 pad 13: /display9/CLK -> CLK
- U30 pad 12: /display10/LOAD -> LOAD
- U30 pad 13: /display10/CLK -> CLK
- U33 pad 12: /display11/LOAD -> LOAD
- U33 pad 13: /display11/CLK -> CLK
- U36 pad 12: /display12/LOAD -> LOAD
- U36 pad 13: /display12/CLK -> CLK
- U39 pad 12: /display13/LOAD -> LOAD
- U39 pad 13: /display13/CLK -> CLK
- U42 pad 12: /display14/LOAD -> LOAD
- U42 pad 13: /display14/CLK -> CLK
- U45 pad 12: /display15/LOAD -> LOAD
- U45 pad 13: /display15/CLK -> CLK
- U48 pad 12: /display16/LOAD -> LOAD
- U48 pad 13: /display16/CLK -> CLK
- U5 pad 12: /display1/LOAD -> LOAD
- U5 pad 13: /display1/CLK -> CLK
- U51 pad 12: /display17/LOAD -> LOAD
- U51 pad 13: /display17/CLK -> CLK
- U54 pad 12: /display18/LOAD -> LOAD
- U54 pad 13: /display18/CLK -> CLK
- U7 pad 15: Net-(U7-Pad15) -> GND
- U7 pad 19: Net-(U7-Pad19) -> CLK
- U7 pad 20: Net-(U7-Pad20) -> /display0/DIN
- U7 pad 6: Net-(U7-Pad6) -> LOAD
- U9 pad 12: /display3/LOAD -> LOAD
- U9 pad 13: /display3/CLK -> CLK
Routing:
- net +5V: track 385.2 -> 1474.4 mm, vias 38 -> 39
- net +3V3: track 0.00 -> 62.5 mm
- net Net-(J1-Pad3): track 0.00 -> 38.8 mm
- net Net-(J1-Pad2): track 0.00 -> 38.6 mm
- net GND: track 145.6 -> 179.5 mm, vias 57 -> 61
- net Net-(R21-Pad2): track 0.00 -> 22.5 mm
- net Net-(R19-Pad1): track 0.00 -> 17.0 mm
- net Net-(R20-Pad2): track 0.00 -> 10.3 mm
- net Net-(R22-Pad2): track 0.00 -> 3.85 mm
- added copper zone on F.Cu, net GND

Commit message: Finished PCB
Routing:
- net LOAD: track 0.00 -> 1384.4 mm, vias 0 -> 25
- net CLK: track 0.00 -> 1384.1 mm, vias 0 -> 25
- net GND: track 179.5 -> 504.5 mm, vias 61 -> 97
- net +5V: track 1474.4 -> 1712.0 mm, vias 39 -> 37
- net /display10/DIN: track 0.00 -> 237.4 mm, vias 0 -> 4
- net /display4/DIN: track 0.00 -> 237.2 mm, vias 0 -> 4
- net /display16/DIN: track 0.00 -> 237.2 mm, vias 0 -> 4
- net /display13/DIN: track 0.00 -> 236.5 mm, vias 0 -> 4
- net /display7/DIN: track 0.00 -> 234.6 mm, vias 0 -> 4
- net /display5/DIN: track 0.00 -> 110.0 mm, vias 0 -> 4
- net /display11/DIN: track 0.00 -> 108.6 mm, vias 0 -> 2
- net /display14/DIN: track 0.00 -> 107.9 mm, vias 0 -> 2
- net /display8/DIN: track 0.00 -> 107.8 mm, vias 0 -> 2
- net /display12/DIN: track 0.00 -> 107.8 mm, vias 0 -> 2
- net /display6/DIN: track 0.00 -> 107.8 mm, vias 0 -> 2
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
Commit message: Added mouting holes
Parts:
- added REF**: MountingHole_3.2mm_M3_Pad, MountingHole:MountingHole_3.2mm_M3_Pad, F.Cu at (259.7, -64.8)
- added REF**: MountingHole_3.2mm_M3_Pad, MountingHole:MountingHole_3.2mm_M3_Pad, F.Cu at (259.7, -162.6)
- added REF**: MountingHole_3.2mm_M3_Pad, MountingHole:MountingHole_3.2mm_M3_Pad, F.Cu at (-26.0, -64.8)
- added REF**: MountingHole_3.2mm_M3_Pad, MountingHole:MountingHole_3.2mm_M3_Pad, F.Cu at (-26.0, -162.6)
Other:
- board text added: "3.3v"
- board text added: "GND"
- board text added: "RX"
- board text added: "TX"
Changed lines of the file:
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@@
   (general
     (thickness 1.6)
-    (drawings 4)
+    (drawings 8)
     (tracks 4051)
     (zones 0)
-    (modules 101)
+    (modules 105)
     (nets 348)
   )
@@
     (0 F.Cu signal)
     (31 B.Cu signal)
-    (32 B.Adhes user)
-    (33 F.Adhes user)
-    (34 B.Paste user)
-    (35 F.Paste user)
-    (36 B.SilkS user)
-    (37 F.SilkS user)
-    (38 B.Mask user)
-    (39 F.Mask user)
-    (40 Dwgs.User user)
-    (41 Cmts.User user)
-    (42 Eco1.User user)
-    (43 Eco2.User user)
-    (44 Edge.Cuts user)
-    (45 Margin user)
-    (46 B.CrtYd user)
-    (47 F.CrtYd user)
-    (48 B.Fab user)
-    (49 F.Fab user)
+    (32 B.Adhes user hide)
+    (33 F.Adhes user hide)
+    (34 B.Paste user hide)
+    (35 F.Paste user hide)
+    (36 B.SilkS user hide)
+    (37 F.SilkS user hide)
+    (38 B.Mask user hide)
+    (39 F.Mask user hide)
+    (40 Dwgs.User user hide)
+    (41 Cmts.User user hide)
+    (42 Eco1.User user hide)
+    (43 Eco2.User user hide)
+    (44 Edge.Cuts user hide)
+    (45 Margin user hide)
+    (46 B.CrtYd user hide)
+    (47 F.CrtYd user hide)
+    (48 B.Fab user hide)
+    (49 F.Fab user hide)
   )
   (setup
@@
     (mod_text_size 1 1)
     (mod_text_width 0.15)
-    (pad_size 1.15 1.4)
-    (pad_drill 0)
+    (pad_size 6.4 6.4)
+    (pad_drill 3.2)
     (pad_to_mask_clearance 0.051)
     (solder_mask_min_width 0.25)
     (aux_axis_origin 0 0)
     (grid_origin -16.51 -154.94)
-    (visible_elements 7FFDFEFF)
+    (visible_elements 7FFFFEFF)
     (pcbplotparams
-      (layerselection 0x010fc_ffffffff)
+      (layerselection 0x010f0_ffffffff)
       (usegerberextensions false)
       (usegerberattributes false)
@@
       (outputformat 1)
       (mirror false)
-      (drillshape 1)
+      (drillshape 0)
       (scaleselection 1)
-      (outputdirectory ""))
+      (outputdirectory "C:/Users/Mattias/Desktop/asdf/"))
   )
   (net 0 "")
@@
     (add_net GND)
   )
+  (module MountingHole:MountingHole_3.2mm_M3_Pad (layer F.Cu)
+    (at 259.715 -64.77)
+    (descr "Mounting Hole 3.2mm, M3")
+    (tags "mounting hole 3.2mm m3")
+    (attr virtual)
+    (fp_text reference REF** (at 0 -4.2) (layer F.SilkS) hide
+      (effects (font (size 1 1) (thickness 0.15)))
+    )
+    (fp_text value MountingHole_3.2mm_M3_Pad (at 0 4.2) (layer F.Fab)
+      (effects (font (size 1 1) (thickness 0.15)))
+    )
+    (fp_circle (center 0 0) (end 3.45 0) (layer F.CrtYd) (width 0.05))
+    (fp_circle (center 0 0) (end 3.2 0) (layer Cmts.User) (width 0.15))
+    (fp_text user %R (at 0.3 0) (layer F.Fab)
+      (effects (font (size 1 1) (thickness 0.15)))
+    )
+    (pad 1 thru_hole circle (at 0 0) (size 6.4 6.4) (drill 3.2) (layers *.Cu *.Mask)
+      (net 2 GND))
+  )
+  (module MountingHole:MountingHole_3.2mm_M3_Pad (layer F.Cu)
+    (at 259.715 -162.56)
+    (descr "Mounting Hole 3.2mm, M3")
+    (tags "mounting hole 3.2mm m3")
+    (attr virtual)
+    (fp_text reference REF** (at 0 -4.2) (layer F.SilkS) hide
+      (effects (font (size 1 1) (thickness 0.15)))
+    )
+    (fp_text value MountingHole_3.2mm_M3_Pad (at 0 4.2) (layer F.Fab)
+      (effects (font (size 1 1) (thickness 0.15)))
+    )
+    (fp_text user %R (at 0.3 0) (layer F.Fab)
+      (effects (font (size 1 1) (thickness 0.15)))
+    )
+    (fp_circle (center 0 0) (end 3.2 0) (layer Cmts.User) (width 0.15))
+    (fp_circle (center 0 0) (end 3.45 0) (layer F.CrtYd) (width 0.05))
+    (pad 1 thru_hole circle (at 0 0) (size 6.4 6.4) (drill 3.2) (layers *.Cu *.Mask)
+      (net 2 GND))
+  )
+  (module MountingHole:MountingHole_3.2mm_M3_Pad (layer F.Cu)
+    (at -26.035 -64.77)
+    (descr "Mounting Hole 3.2mm, M3")
+    (tags "mounting hole 3.2mm m3")
+    (attr virtual)
+    (fp_text reference REF** (at 0 -4.2) (layer F.SilkS) hide
+      (effects (font (size 1 1) (thickness 0.15)))
+    )
+    (fp_text value MountingHole_3.2mm_M3_Pad (at 0 4.2) (layer F.Fab)
+      (effects (font (size 1 1) (thickness 0.15)))
+    )
+    (fp_text user %R (at 0.3 0) (layer F.Fab)
+      (effects (font (size 1 1) (thickness 0.15)))
+    )
+    (fp_circle (center 0 0) (end 3.2 0) (layer Cmts.User) (width 0.15))
+    (fp_circle (center 0 0) (end 3.45 0) (layer F.CrtYd) (width 0.05))
+    (pad 1 thru_hole circle (at 0 0) (size 6.4 6.4) (drill 3.2) (layers *.Cu *.Mask)
+      (net 2 GND))
+  )
+  (module MountingHole:MountingHole_3.2mm_M3_Pad (layer F.Cu)
+    (at -26.035 -162.56)
+    (descr "Mounting Hole 3.2mm, M3")
+    (tags "mounting hole 3.2mm m3")
+    (attr virtual)
+    (fp_text reference REF** (at 0 -4.2) (layer F.SilkS) hide
+      (effects (font (size 1 1) (thickness 0.15)))
+    )
+    (fp_text value MountingHole_3.2mm_M3_Pad (at 0 4.2) (layer F.Fab)
+      (effects (font (size 1 1) (thickness 0.15)))
+    )
+    (fp_circle (center 0 0) (end 3.45 0) (layer F.CrtYd) (width 0.05))
+    (fp_circle (center 0 0) (end 3.2 0) (layer Cmts.User) (width 0.15))
+    (fp_text user %R (at 0.3 0) (layer F.Fab)
+      (effects (font (size 1 1) (thickness 0.15)))
+    )
+    (pad 1 thru_hole circle (at 0 0) (size 6.4 6.4) (drill 3.2) (layers *.Cu *.Mask)
+      (net 2 GND))
+  )
   (module circuit:7seg (layer F.Cu)
     (at -16.51 -57.15 90)
@@
     (descr "4 digit 7 segment green LED, http://www.kingbright.com/attachments/file/psearch/000/00/00/CA56-12CGKWA(Ver.9A).pdf")
     (tags "4 digit 7 segment green LED")
-    (fp_text reference U14 (at 0.195 -17.61 90) (layer F.SilkS)
+    (fp_text reference U14 (at 0.195 -17.61 90) (layer F.SilkS) hide
       (effects (font (size 1 1) (thickness 0.15)))
     )
@@
     (tags "SPST button tactile switch")
     (attr smd)
-    (fp_text reference SW1 (at 0 2.6 180) (layer B.SilkS)
+    (fp_text reference SW1 (at 0 -3.175 180) (layer B.SilkS)
       (effects (font (size 1 1) (thickness 0.15)) (justify mirror))
     )
-    (fp_text value Reset (at 0 -3 180) (layer B.SilkS)
+    (fp_text value Reset (at 0 3.175 180) (layer B.SilkS)
       (effects (font (size 1 1) (thickness 0.15)) (justify mirror))
     )
@@
     )
   )
+  (gr_text 3.3v (at 62.23 -132.715 90) (layer B.SilkS)
+    (effects (font (size 1 1) (thickness 0.15)) (justify mirror))
+  )
+  (gr_text RX (at 64.77 -133.35 90) (layer B.SilkS)
+    (effects (font (size 1 1) (thickness 0.15)) (justify mirror))
+  )
+  (gr_text TX (at 67.31 -133.35 90) (layer B.SilkS)
+    (effects (font (size 1 1) (thickness 0.15)) (justify mirror))
+  )
+  (gr_text GND (at 69.85 -132.715 90) (layer B.SilkS)
+    (effects (font (size 1 1) (thickness 0.15)) (justify mirror))
+  )
   (gr_line (start -35.56 -54.991) (end -35.56 -172.339) (layer Edge.Cuts) (width 0.05))
   (gr_line (start 269.24 -54.991) (end -35.56 -54.991) (layer Edge.Cuts) (width 0.05))
   (gr_line (start 269.24 -172.339) (end 269.24 -54.991) (layer Edge.Cuts) (width 0.05))
   (gr_line (start -35.56 -172.339) (end 269.24 -172.339) (layer Edge.Cuts) (width 0.05))
-  (via (at 158.75 -138.43) (size 0.8) (drill 0.4) (layers F.Cu B.Cu) (net 2))
-  (via (at 151.13 -138.43) (size 0.8) (drill 0.4) (layers F.Cu B.Cu) (net 2))
-  (segment (start 151.13 -138.43) (end 158.75 -138.43) (width 0.5) (layer B.Cu) (net 2))
-  (via (at 158.75 -117.475) (size 0.8) (drill 0.4) (layers F.Cu B.Cu) (net 2))
-  (via (at 151.13 -117.475) (size 0.8) (drill 0.4) (layers F.Cu B.Cu) (net 2))
-  (segment (start 151.13 -117.475) (end 158.75 -117.475) (width 0.5) (layer B.Cu) (net 2))
-  (via (at 158.115 -98.425) (size 0.8) (drill 0.4) (layers F.Cu B.Cu) (net 2))
-  (via (at 150.495 -98.425) (size 0.8) (drill 0.4) (layers F.Cu B.Cu) (net 2))
-  (segment (start 150.495 -98.425) (end 158.115 -98.425) (width 0.5) (layer B.Cu) (net 2))
-  (via (at 158.75 -78.74) (size 0.8) (drill 0.4) (layers F.Cu B.Cu) (net 2))
-  (via (at 151.13 -78.74) (size 0.8) (drill 0.4) (layers F.Cu B.Cu) (net 2))
-  (segment (start 151.13 -78.74) (end 158.75 -78.74) (width 0.5) (layer B.Cu) (net 2))
-  (via (at 52.07 -166.37) (size 0.8) (drill 0.4) (layers F.Cu B.Cu) (net 2))
-  (via (at 167.64 -151.765) (size 0.8) (drill 0.4) (layers F.Cu B.Cu) (net 2))
-  (via (at 167.64 -168.275) (size 0.8) (drill 0.4) (layers F.Cu B.Cu) (net 2))
   (segment (start 117.865 -111.506) (end 117.865 -110.806) (width 0.25) (layer B.Cu) (net 1) (status 10))
   (segment (start 117.475 -104.521) (end 128.905 -104.521) (width 0.5) (layer F.Cu) (net 1))
@@
   (segment (start 218.99499 -167.12999) (end 219.075 -167.21) (width 0.5) (layer B.Cu) (net 1) (status 30))
   (segment (start 218.99499 -164.465) (end 218.99499 -167.12999) (width 0.5) (layer B.Cu) (net 1) (status 20))
+  (via (at 158.75 -138.43) (size 0.8) (drill 0.4) (layers F.Cu B.Cu) (net 2))
+  (via (at 151.13 -138.43) (size 0.8) (drill 0.4) (layers F.Cu B.Cu) (net 2))
+  (segment (start 151.13 -138.43) (end 158.75 -138.43) (width 0.5) (layer B.Cu) (net 2))
+  (via (at 158.75 -117.475) (size 0.8) (drill 0.4) (layers F.Cu B.Cu) (net 2))
+  (via (at 151.13 -117.475) (size 0.8) (drill 0.4) (layers F.Cu B.Cu) (net 2))
+  (segment (start 151.13 -117.475) (end 158.75 -117.475) (width 0.5) (layer B.Cu) (net 2))
+  (via (at 158.115 -98.425) (size 0.8) (drill 0.4) (layers F.Cu B.Cu) (net 2))
+  (via (at 150.495 -98.425) (size 0.8) (drill 0.4) (layers F.Cu B.Cu) (net 2))
+  (segment (start 150.495 -98.425) (end 158.115 -98.425) (width 0.5) (layer B.Cu) (net 2))
+  (via (at 158.75 -78.74) (size 0.8) (drill 0.4) (layers F.Cu B.Cu) (net 2))
+  (via (at 151.13 -78.74) (size 0.8) (drill 0.4) (layers F.Cu B.Cu) (net 2))
+  (segment (start 151.13 -78.74) (end 158.75 -78.74) (width 0.5) (layer B.Cu) (net 2))
+  (via (at 52.07 -166.37) (size 0.8) (drill 0.4) (layers F.Cu B.Cu) (net 2))
+  (via (at 167.64 -151.765) (size 0.8) (drill 0.4) (layers F.Cu B.Cu) (net 2))
+  (via (at 167.64 -168.275) (size 0.8) (drill 0.4) (layers F.Cu B.Cu) (net 2))
   (via (at 118.11 -101.346) (size 0.8) (drill 0.4) (layers F.Cu B.Cu) (net 2))
   (via (at 114.935 -101.346) (size 0.8) (drill 0.4) (layers F.Cu B.Cu) (net 2))
