File: circuit/7-seg-array-clock.kicad_pcb (KiCad board)
At the start: 2 copper layers, 304.8 x 117.3 mm, 106 parts, among them J1 FTDI, J2 USB_B_Mini, SW1 Reset, SW2 Flash, U1 CC56-12EWA, U10 CC56-12EWA, U11 CC56-12EWA, U12 MAX7219, U13 CC56-12EWA, U14 CC56-12EWA, U15 MAX7219, U16 CC56-12EWA, U17 CC56-12EWA, U18 MAX7219, U19 CC56-12EWA, U2 MAX7219, U20 CC56-12EWA, U21 MAX7219, U22 CC56-12EWA, U23 CC56-12EWA, U24 MAX7219, U25 CC56-12EWA, U26 CC56-12EWA, U27 MAX7219, U28 CC56-12EWA, U29 CC56-12EWA, U3 CC56-12EWA, U30 MAX7219, U31 CC56-12EWA, U32 CC56-12EWA, U33 MAX7219, U34 CC56-12EWA, U35 CC56-12EWA, U36 MAX7219, U37 CC56-12EWA, U38 CC56-12EWA, U39 MAX7219, U4 CC56-12EWA, U40 CC56-12EWA, U41 CC56-12EWA, U42 MAX7219, U43 CC56-12EWA, U44 CC56-12EWA, U45 MAX7219, U46 CC56-12EWA, U47 CC56-12EWA, U48 MAX7219, U49 CC56-12EWA, U5 MAX7219, U50 CC56-12EWA, U51 MAX7219, U52 CC56-12EWA, U53 CC56-12EWA, U54 MAX7219, U55 CC56-12EWA, U56 LM1117-3.3, U6 CC56-12EWA, U7 ESP-12F, U8 CC56-12EWA, U9 MAX7219

Commit message: Moved components
Parts:
- moved C5 194.3 mm to (160.8, 48.1)
- moved SW1 178.4 mm to (118.6, 10.6)
- moved R1 176.0 mm to (50.4, 2.25)
- moved C1 175.8 mm to (59.9, 9.63)
- moved R2 175.8 mm to (151.3, 2.25)
- moved REF** 175.8 mm to (9.62, 9.62)
- moved U7 175.8 mm to (100.9, 12.2)
- moved U1 175.8 mm to (18.9, 17.2)
- moved C19 175.8 mm to (89.6, 51.6)
- moved C20 175.8 mm to (89.6, 55.6)
- moved R21 175.8 mm to (102.6, 33.2)
- moved SW2 175.8 mm to (97.9, 29.4)
- moved U56 175.8 mm to (97.9, 53.5)
- moved J1 175.8 mm to (94.1, 37.0)
- moved U2 175.8 mm to (50.4, 9.63)
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Routing:
- net /display4/F: track 55.3 -> 83.0 mm
- net /display4/DP: track 81.6 -> 53.9 mm
Other:
- board size 304.8 x 117.3 mm -> 302.6 x 115.4 mm

Commit message: Routed first 8 digits
Parts:
- moved C5 19.2 mm to (160.8, 28.9)
- moved R15 19.2 mm to (252.2, 79.2)
Routing:
- net +5V: track 1719.4 -> 7.60 mm, vias 38 -> 1
- net LOAD: track 1390.1 -> 0.00 mm, vias 25 -> 0
- net CLK: track 1386.1 -> 0.00 mm, vias 25 -> 0
- net GND: track 505.3 -> 6.20 mm, vias 103 -> 2
- net /display10/DIN: track 237.4 -> 0.00 mm, vias 4 -> 0
- net /display4/DIN: track 237.2 -> 0.00 mm, vias 4 -> 0
- net /display16/DIN: track 237.2 -> 0.00 mm, vias 4 -> 0
- net /display13/DIN: track 236.5 -> 0.00 mm, vias 4 -> 0
- net /display7/DIN: track 234.6 -> 0.00 mm, vias 4 -> 0
- net /display5/DIN: track 110.0 -> 0.00 mm, vias 4 -> 0
- net /display11/DIN: track 108.6 -> 0.00 mm, vias 2 -> 0
- net /display14/DIN: track 107.9 -> 0.00 mm, vias 2 -> 0
- net /display8/DIN: track 107.8 -> 0.00 mm, vias 2 -> 0
- net /display12/DIN: track 107.8 -> 0.00 mm, vias 2 -> 0
- net /display6/DIN: track 107.8 -> 0.00 mm, vias 2 -> 0
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- removed copper zone on B.Cu, net GND

Commit message: Copied tracks to other displays
Routing:
- net +5V: track 7.60 -> 186.2 mm, vias 1 -> 36
- net GND: track 6.20 -> 144.8 mm, vias 2 -> 54
- net /display9/G: track 0.00 -> 82.0 mm
- net /display6/G: track 0.00 -> 82.0 mm
- net /display3/G: track 0.00 -> 82.0 mm
- net /display18/G: track 0.00 -> 82.0 mm
- net /display12/G: track 0.00 -> 82.0 mm
- net /display15/G: track 0.00 -> 82.0 mm
- net /display8/G: track 0.00 -> 82.0 mm
- net /display7/G: track 0.00 -> 82.0 mm
- net /display5/G: track 0.00 -> 82.0 mm
- net /display4/G: track 0.00 -> 82.0 mm
- net /display17/G: track 0.00 -> 82.0 mm
- net /display16/G: track 0.00 -> 82.0 mm
- net /display13/G: track 0.00 -> 82.0 mm
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
Commit message: Finished board with proper spacing
Parts:
- moved J1 26.5 mm to (87.0, 11.4), turned to 180 degrees
- moved SW1 21.9 mm to (109.2, 30.4), turned to 270 degrees
- moved R21 11.4 mm to (92.7, 27.6), turned to 90 degrees
- moved SW2 9.05 mm to (88.9, 30.4), turned to 270 degrees
- moved R22 6.22 mm to (90.6, 21.7)
- moved R19 5.67 mm to (111.9, 18.7), turned to 90 degrees
- moved R20 4.40 mm to (111.9, 13.8)
- moved U56 1.53 mm to (98.5, 52.1)
Routing:
- net +5V: track 186.2 -> 1671.2 mm, vias 36 -> 45
- net LOAD: track 81.6 -> 1434.4 mm, vias 18 -> 24
- net CLK: track 57.2 -> 1378.6 mm, vias 18 -> 25
- net /display7/DIN: track 0.00 -> 237.0 mm, vias 0 -> 2
- net /display4/DIN: track 0.00 -> 237.0 mm, vias 0 -> 2
- net /display16/DIN: track 0.00 -> 237.0 mm, vias 0 -> 2
- net /display13/DIN: track 0.00 -> 237.0 mm, vias 0 -> 2
- net /display10/DIN: track 0.00 -> 237.0 mm, vias 0 -> 2
- net /display9/DIN: track 0.00 -> 107.2 mm, vias 0 -> 2
- net /display8/DIN: track 0.00 -> 107.2 mm, vias 0 -> 2
- net /display6/DIN: track 0.00 -> 107.2 mm, vias 0 -> 2
- net /display5/DIN: track 0.00 -> 107.2 mm, vias 0 -> 2
- net /display3/DIN: track 0.00 -> 107.2 mm, vias 0 -> 2
- net /display17/DIN: track 0.00 -> 107.2 mm, vias 0 -> 2
- net /display15/DIN: track 0.00 -> 107.2 mm, vias 0 -> 2
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- added copper zone on B.Cu, net GND
