File: circuit/7-seg-array-clock.kicad_pcb (KiCad board)
At the start: 2 copper layers, 302.6 x 115.4 mm, 106 parts, among them J1 FTDI, J2 USB_B_Mini, SW1 Reset, SW2 Flash, U1 CC56-12EWA, U10 CC56-12EWA, U11 CC56-12EWA, U12 MAX7219, U13 CC56-12EWA, U14 CC56-12EWA, U15 MAX7219, U16 CC56-12EWA, U17 CC56-12EWA, U18 MAX7219, U19 CC56-12EWA, U2 MAX7219, U20 CC56-12EWA, U21 MAX7219, U22 CC56-12EWA, U23 CC56-12EWA, U24 MAX7219, U25 CC56-12EWA, U26 CC56-12EWA, U27 MAX7219, U28 CC56-12EWA, U29 CC56-12EWA, U3 CC56-12EWA, U30 MAX7219, U31 CC56-12EWA, U32 CC56-12EWA, U33 MAX7219, U34 CC56-12EWA, U35 CC56-12EWA, U36 MAX7219, U37 CC56-12EWA, U38 CC56-12EWA, U39 MAX7219, U4 CC56-12EWA, U40 CC56-12EWA, U41 CC56-12EWA, U42 MAX7219, U43 CC56-12EWA, U44 CC56-12EWA, U45 MAX7219, U46 CC56-12EWA, U47 CC56-12EWA, U48 MAX7219, U49 CC56-12EWA, U5 MAX7219, U50 CC56-12EWA, U51 MAX7219, U52 CC56-12EWA, U53 CC56-12EWA, U54 MAX7219, U55 CC56-12EWA, U56 LM1117-3.3, U6 CC56-12EWA, U7 ESP-12F, U8 CC56-12EWA, U9 MAX7219

Commit message: Added logo to PCB
Parts:
- added REF**: logo, circuit:logo, B.Cu at (98.8, 104.5)

Commit message: Added voltage test pads
Parts:
- added REF**: TestPoint_Pad_D3.0mm, TestPoint:TestPoint_Pad_D3.0mm, B.Cu at (95.2, 66.0)
- added REF**: TestPoint_Pad_D3.0mm, TestPoint:TestPoint_Pad_D3.0mm, B.Cu at (90.2, 66.0)
- added REF**: TestPoint_Pad_D3.0mm, TestPoint:TestPoint_Pad_D3.0mm, B.Cu at (290.8, 66.0)
- added REF**: TestPoint_Pad_D3.0mm, TestPoint:TestPoint_Pad_D3.0mm, B.Cu at (290.8, 71.1)
Routing:
- net GND: track 163.7 -> 206.6 mm, vias 61 -> 64
- net +5V: track 1671.2 -> 1687.6 mm
- net +3V3: track 98.8 -> 108.4 mm
Other:
- board text added: "5v"
Changed lines of the file:
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@@
   (general
     (thickness 1.6)
-    (drawings 8)
-    (tracks 4109)
+    (drawings 12)
+    (tracks 4126)
     (zones 0)
-    (modules 107)
+    (modules 111)
     (nets 350)
   )
@@
     (mod_text_size 1 1)
     (mod_text_width 0.15)
-    (pad_size 6.4 6.4)
-    (pad_drill 3.2)
+    (pad_size 3 3)
+    (pad_drill 0)
     (pad_to_mask_clearance 0.051)
     (solder_mask_min_width 0.25)
@@
     (add_net GND)
   )
+  (module TestPoint:TestPoint_Pad_D3.0mm (layer B.Cu)
+    (at 95.25 66.04)
+    (descr "SMD pad as test Point, diameter 3.0mm")
+    (tags "test point SMD pad")
+    (attr virtual)
+    (fp_text reference REF** (at 0 2.398) (layer B.SilkS) hide
+      (effects (font (size 1 1) (thickness 0.15)) (justify mirror))
+    )
+    (fp_text value TestPoint_Pad_D3.0mm (at 0 -2.55) (layer B.Fab)
+      (effects (font (size 1 1) (thickness 0.15)) (justify mirror))
+    )
+    (fp_circle (center 0 0) (end 0 -1.75) (layer B.SilkS) (width 0.12))
+    (fp_circle (center 0 0) (end 2 0) (layer B.CrtYd) (width 0.05))
+    (fp_text user %R (at 0 2.4) (layer B.Fab)
+      (effects (font (size 1 1) (thickness 0.15)) (justify mirror))
+    )
+    (pad 1 smd circle (at 0 0) (size 3 3) (layers B.Cu B.Mask)
+      (net 2 GND))
+  )
+  (module TestPoint:TestPoint_Pad_D3.0mm (layer B.Cu)
+    (at 90.17 66.04)
+    (descr "SMD pad as test Point, diameter 3.0mm")
+    (tags "test point SMD pad")
+    (attr virtual)
+    (fp_text reference REF** (at 0 2.398) (layer B.SilkS) hide
+      (effects (font (size 1 1) (thickness 0.15)) (justify mirror))
+    )
+    (fp_text value TestPoint_Pad_D3.0mm (at 0 -2.55) (layer B.Fab)
+      (effects (font (size 1 1) (thickness 0.15)) (justify mirror))
+    )
+    (fp_circle (center 0 0) (end 0 -1.75) (layer B.SilkS) (width 0.12))
+    (fp_circle (center 0 0) (end 2 0) (layer B.CrtYd) (width 0.05))
+    (fp_text user %R (at 0 2.4) (layer B.Fab)
+      (effects (font (size 1 1) (thickness 0.15)) (justify mirror))
+    )
+    (pad 1 smd circle (at 0 0) (size 3 3) (layers B.Cu B.Mask)
+      (net 58 +3V3))
+  )
+  (module TestPoint:TestPoint_Pad_D3.0mm (layer B.Cu)
+    (at 290.83 66.04)
+    (descr "SMD pad as test Point, diameter 3.0mm")
+    (tags "test point SMD pad")
+    (attr virtual)
+    (fp_text reference REF** (at 0 2.398) (layer B.SilkS) hide
+      (effects (font (size 1 1) (thickness 0.15)) (justify mirror))
+    )
+    (fp_text value TestPoint_Pad_D3.0mm (at 0 -2.55) (layer B.Fab)
+      (effects (font (size 1 1) (thickness 0.15)) (justify mirror))
+    )
+    (fp_circle (center 0 0) (end 0 -1.75) (layer B.SilkS) (width 0.12))
+    (fp_circle (center 0 0) (end 2 0) (layer B.CrtYd) (width 0.05))
+    (fp_text user %R (at 0 2.4) (layer B.Fab)
+      (effects (font (size 1 1) (thickness 0.15)) (justify mirror))
+    )
+    (pad 1 smd circle (at 0 0) (size 3 3) (layers B.Cu B.Mask)
+      (net 2 GND))
+  )
+  (module TestPoint:TestPoint_Pad_D3.0mm (layer B.Cu)
+    (at 290.83 71.12)
+    (descr "SMD pad as test Point, diameter 3.0mm")
+    (tags "test point SMD pad")
+    (attr virtual)
+    (fp_text reference REF** (at 0 2.398) (layer B.SilkS) hide
+      (effects (font (size 1 1) (thickness 0.15)) (justify mirror))
+    )
+    (fp_text value TestPoint_Pad_D3.0mm (at 0 -2.55) (layer B.Fab)
+      (effects (font (size 1 1) (thickness 0.15)) (justify mirror))
+    )
+    (fp_circle (center 0 0) (end 0 -1.75) (layer B.SilkS) (width 0.12))
+    (fp_circle (center 0 0) (end 2 0) (layer B.CrtYd) (width 0.05))
+    (fp_text user %R (at 0 2.4) (layer B.Fab)
+      (effects (font (size 1 1) (thickness 0.15)) (justify mirror))
+    )
+    (pad 1 smd circle (at 0 0) (size 3 3) (layers B.Cu B.Mask)
+      (net 1 +5V))
+  )
   (module circuit:logo (layer B.Cu)
     (at 98.8314 104.521 180)
@@
       (effects (font (size 1 1) (thickness 0.15)) (justify mirror))
     )
-    (fp_text value logo (at 7.62 -7.62) (layer B.Fab)
+    (fp_text value logo (at 7.62 -7.62) (layer B.Fab) hide
       (effects (font (size 1 1) (thickness 0.15)) (justify mirror))
     )
@@
     )
   )
+  (gr_text 5v (at 295.402 71.374) (layer B.SilkS)
+    (effects (font (size 1.5 1.5) (thickness 0.3)) (justify mirror))
+  )
+  (gr_text GND (at 295.402 66.04) (layer B.SilkS)
+    (effects (font (size 1.5 1.5) (thickness 0.3)) (justify mirror))
+  )
+  (gr_text GND (at 99.822 66.04) (layer B.SilkS)
+    (effects (font (size 1.5 1.5) (thickness 0.3)) (justify mirror))
+  )
+  (gr_text 3.3v (at 85.598 66.04) (layer B.SilkS)
+    (effects (font (size 1.5 1.5) (thickness 0.3)) (justify mirror))
+  )
   (gr_line (start 302.64 0) (end 302.64 115.44) (layer Edge.Cuts) (width 0.05))
   (gr_line (start 0 115.44) (end 302.64 115.44) (layer Edge.Cuts) (width 0.05))
@@
   (via (at 282.194 84.963) (size 0.8) (drill 0.4) (layers F.Cu B.Cu) (net 1))
   (segment (start 293.573 84.963) (end 293.59 84.98) (width 0.5) (layer B.Cu) (net 1))
-  (segment (start 282.194 84.963) (end 293.573 84.963) (width 0.5) (layer B.Cu) (net 1))
   (segment (start 202.311 9.525) (end 263.99 9.525) (width 0.5) (layer F.Cu) (net 1))
   (via (at 201.76 9.525) (size 0.8) (drill 0.4) (layers F.Cu B.Cu) (net 1))
@@
   (segment (start 92.33 49.6808) (end 92.33 48.005) (width 0.5) (layer B.Cu) (net 1))
   (segment (start 92.4192 49.77) (end 92.33 49.6808) (width 0.5) (layer B.Cu) (net 1))
+  (segment (start 284.607 84.963) (end 284.607 82.423) (width 0.5) (layer B.Cu) (net 1))
+  (segment (start 284.607 84.963) (end 293.573 84.963) (width 0.5) (layer B.Cu) (net 1))
+  (segment (start 282.194 84.963) (end 284.607 84.963) (width 0.5) (layer B.Cu) (net 1))
+  (segment (start 284.607 82.423) (end 290.83 76.2) (width 0.5) (layer B.Cu) (net 1))
+  (segment (start 290.83 76.2) (end 290.83 71.12) (width 0.5) (layer B.Cu) (net 1))
   (via (at 51.816 11.811) (size 0.8) (drill 0.4) (layers F.Cu B.Cu) (net 2))
   (segment (start 53.615 14.28) (end 53.615 13.61) (width 0.5) (layer B.Cu) (net 2))
@@
   (via (at 109.22 36.957) (size 0.8) (drill 0.4) (layers F.Cu B.Cu) (net 2))
   (segment (start 109.22 34.29) (end 109.22 36.957) (width 0.5) (layer B.Cu) (net 2))
+  (segment (start 290.83 66.04) (end 293.37 66.04) (width 0.5) (layer B.Cu) (net 2))
+  (segment (start 293.37 66.04) (end 295.91 68.58) (width 0.5) (layer B.Cu) (net 2))
+  (segment (start 295.91 68.58) (end 295.91 81.28) (width 0.5) (layer B.Cu) (net 2))
+  (via (at 285.75 66.04) (size 0.8) (drill 0.4) (layers F.Cu B.Cu) (net 2))
+  (segment (start 290.83 66.04) (end 285.75 66.04) (width 0.5) (layer B.Cu) (net 2))
+  (segment (start 290.83 66.04) (end 290.83 63.5) (width 0.5) (layer B.Cu) (net 2))
+  (via (at 290.83 60.96) (size 0.8) (drill 0.4) (layers F.Cu B.Cu) (net 2))
+  (segment (start 290.83 63.5) (end 290.83 60.96) (width 0.5) (layer B.Cu) (net 2))
+  (segment (start 95.25 66.04) (end 95.25 57.15) (width 0.5) (layer B.Cu) (net 2))
+  (via (at 95.25 71.12) (size 0.8) (drill 0.4) (layers F.Cu B.Cu) (net 2))
+  (segment (start 95.25 66.04) (end 95.25 71.12) (width 0.5) (layer B.Cu) (net 2))
   (segment (start 49.805 3.955) (end 49.805 4.98) (width 0.25) (layer B.Cu) (net 3))
   (segment (start 49.805 3.34) (end 49.805 3.955) (width 0.25) (layer B.Cu) (net 3))
@@
   (segment (start 86.995 11.43) (end 95.561685 11.43) (width 0.5) (layer F.Cu) (net 58))
   (via (at 100.871 16.891) (size 0.8) (drill 0.4) (layers F.Cu B.Cu) (net 58))
+  (segment (start 90.17 57.2064) (end 89.6344 56.6708) (width 0.5) (layer B.Cu) (net 58))
+  (segment (start 90.17 66.04) (end 90.17 57.2064) (width 0.5) (layer B.Cu) (net 58))
   (segment (start 264.498 17.272) (end 264.476 17.25) (width 0.25) (layer B.Cu) (net 66))
   (segment (start 260.053 11.55559) (end 260.053 12.827) (width 0.25) (layer B.Cu) (net 66))
